File: blocks/24_to_5_supply.sch (KiCad schematic (older format))
At the start: 0 parts

Commit message: added multiple schematics
Parts:
- added C? (x2): 1u, symbol Device:C
- added C?: 100n, symbol Device:C
- added D?: D_Schottky, symbol Device:D_Schottky
- added D? (x2): D_TVS, symbol Device:D_TVS
- added F?: Fuse, symbol Device:Fuse
- added FB?: Ferrite_Bead, symbol Device:Ferrite_Bead
- added VR?: Wurth-FDSM, KTHFS:Wurth-FDSM, symbol KTHFS:Wurth-FDSM
Connections:
- new net: FB?.2, VR?.3 (OUT)
- new net: D?.1 (K), F?.2
- new net +24V: C?.1, D?.1 (A1), F?.1, VR?.1 (IN)
- new net +5V: C?.1, C?.1, D?.1 (A1), FB?.1
- new net GND: C?.2, C?.2, C?.2, D?.2 (A2), D?.2 (A2), VR?.2 (GND)
- new net battery_in: D?.2 (A)
Other:
- note added: "tells ERC that this is\na power source"
